Commit message: Add kuromitsu settings

File: ros/kxr_models/urdf/kuromitsu.urdf (robot description, URDF)
Before this commit: robot kuromitsu, 13 links, 12 joints
Links:
- link LLEG_LINK0: geometry collision cylinder length=0.01 radius=0.05; visual mesh filename=package://kxr_models/meshes/kuromitsu/LLEG_LINK0_mesh.dae scale=1 1 1
- link LLEG_LINK1: geometry collision cylinder length=0.01 radius=0.05; visual mesh filename=package://kxr_models/meshes/kuromitsu/LLEG_LINK1_mesh.dae scale=1 1 1
- link RLEG_LINK0: geometry collision cylinder length=0.01 radius=0.05; visual mesh filename=package://kxr_models/meshes/kuromitsu/RLEG_LINK0_mesh.dae scale=1 1 1
- link RLEG_LINK1: geometry collision cylinder length=0.01 radius=0.05; visual mesh filename=package://kxr_models/meshes/kuromitsu/RLEG_LINK1_mesh.dae scale=1 1 1
Joints:
- joint HEAD_JOINT0: axis 0 0 1 -> 0 0 -1
- joint HEAD_JOINT1: axis 0 1 0 -> 0 -1 0
- joint LARM_JOINT0: axis 0 1 0 -> 0 -1 0
- joint LARM_JOINT1: axis 1 0 0 -> -1 0 0
- joint LARM_JOINT2: axis 0 1 0 -> 0 -1 0

Commit message: Loose joint limit for demo

File: ros/kxr_models/urdf/kuromitsu.urdf (robot description, URDF)
Before this commit: robot kuromitsu, 13 links, 12 joints
Joints:
- joint HEAD_JOINT0: limit lower=-2.96706 upper=2.96706 effort=0.656248 velocity=7.47998 -> lower=-20.96706 upper=20.96706 effort=0.656248 velocity=7.47998
- joint HEAD_JOINT1: limit lower=-2.0944 upper=2.0944 effort=0.656248 velocity=7.47998 -> lower=-20.0944 upper=20.0944 effort=0.656248 velocity=7.47998
- joint LARM_JOINT0: limit lower=-3.14159 upper=3.14159 effort=0.656248 velocity=7.47998 -> lower=-30.14159 upper=30.14159 effort=0.656248 velocity=7.47998
- joint LARM_JOINT1: limit lower=-0.523599 upper=3.22886 effort=0.656248 velocity=7.47998 -> lower=-30.523599 upper=30.22886 effort=0.656248 velocity=7.47998
- joint LARM_JOINT2: limit lower=-2.96706 upper=2.96706 effort=0.656248 velocity=7.47998 -> lower=-20.96706 upper=20.96706 effort=0.656248 velocity=7.47998
- joint RARM_JOINT0: limit lower=-3.14159 upper=3.14159 effort=0.656248 velocity=7.47998 -> lower=-30.14159 upper=30.14159 effort=0.656248 velocity=7.47998
- joint RARM_JOINT1: limit lower=-3.22886 upper=0.523599 effort=0.656248 velocity=7.47998 -> lower=-30.22886 upper=30.523599 effort=0.656248 velocity=7.47998
- joint RARM_JOINT2: limit lower=-2.96706 upper=2.96706 effort=0.656248 velocity=7.47998 -> lower=-20.96706 upper=20.96706 effort=0.656248 velocity=7.47998
