Commit message: Add kashiwagi

File: ros/kxr_models/urdf/kashiwagi.urdf (robot description, URDF)
Before this commit: robot kashiwagi, 11 links, 10 joints
Links:
- link LLEG_LINK0: geometry collision cylinder length=0.01 radius=0.05; visual mesh filename=package://kxr_models/meshes/kashiwagi/LLEG_LINK0_mesh.dae scale=1 1 1
- link LLEG_LINK1: geometry collision cylinder length=0.01 radius=0.05; visual mesh filename=package://kxr_models/meshes/kashiwagi/LLEG_LINK1_mesh.dae scale=1 1 1
- link RLEG_LINK0: geometry collision cylinder length=0.01 radius=0.05; visual mesh filename=package://kxr_models/meshes/kashiwagi/RLEG_LINK0_mesh.dae scale=1 1 1
- link RLEG_LINK1: geometry collision cylinder length=0.01 radius=0.05; visual mesh filename=package://kxr_models/meshes/kashiwagi/RLEG_LINK1_mesh.dae scale=1 1 1

Commit message: Loose

File: ros/kxr_models/urdf/kashiwagi.urdf (robot description, URDF)
Before this commit: robot kashiwagi, 11 links, 10 joints
Joints:
- joint LARM_JOINT1: limit lower=-0.523599 upper=3.22886 effort=0.656248 velocity=7.47998 -> lower=-10 upper=10 effort=0.656248 velocity=7.47998
- joint RARM_JOINT1: limit lower=-3.22886 upper=0.523599 effort=0.656248 velocity=7.47998 -> lower=-10 upper=10 effort=0.656248 velocity=7.47998
